File: PXF_CAPE_PCB/PixHawk_Fire_v1.2.brd (EAGLE design)
At the start: 86.4 x 54.6 mm, 242 parts, among them J305 DF13-3P-1.25V, J306 DF13-4P-1.25V, J307 DF13-4P-1.25V, J308 DF13-4P-1.25V, J309 DF13-5P-1.25V, J310 DF13-4P-1.25V, J314 DF13-4P-1.25V, J701 JST-ZH-3, J801 DF13C-6P-1.25V, M3_MOUNT901 MOUNT-HOLE3.1MM, M3_MOUNT902 MOUNT-HOLE3.1MM, M3_MOUNT903 MOUNT-HOLE3.1MM, M3_MOUNT904 MOUNT-HOLE3.1MM, Q501 MMBT3906LT1SMD, U1 EEPROM-I2CSMD, U102 FM25V01, U2 EEPROM-I2CSMD, U201 TXS0108QFN20, U202 TXS0108QFN20, U301 MAX3051, U302 TXS0108QFN20, U303 PCA9306, U401 MS5611-01BA, U402 MS5611-01BA, U403 MPU-6000, U405 MPU-9250, U406 LSM9DS0LSM9DS0, U407 BMP280_PRELIM, U501 BQ24315, U502 MIC5332, U503 BQ24315, U601 TCA62724FMG, U602 LT3469, U603 LRTB GFTG-T7AW-1+V7A7-29+R5T9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, U701 TXS0108QFN20, U702 TXS0108QFN20, U703 74LVC2G240, U704 BBB_3X14_RA, U801 BQ24313, U802 MIC5332, X801 4 pin head

Commit message: Fixes in some typos with components
Parts:
- C409, C414: value 2200p -> 0u1
Changed lines of the file:
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@@
 <attribute name="PARTNO" value="MPU-6000" x="126.6792" y="27.2836" size="1.778" layer="28" rot="MR0" display="off"/>
 </element>
-<element name="C409" library="pixhawk2" package="0603-CAP" value="2200p" x="127.816" y="22.6992" rot="MR180">
+<element name="C409" library="pixhawk2" package="0603-CAP" value="0u1" x="127.816" y="22.6992" rot="MR180">
 <attribute name="PARTNO" value="C0603C222J5RACTU" x="127.816" y="22.6992" size="1.778" layer="28" rot="MR180" display="off"/>
 </element>
@@
 <attribute name="PARTNO" value="MCR01MRTF1004" x="144.5216" y="33.614" size="1.778" layer="28" rot="MR0" display="off"/>
 </element>
-<element name="C414" library="pixhawk2" package="0402-CAP" value="2200p" x="124.9396" y="20.9496" rot="MR0">
+<element name="C414" library="pixhawk2" package="0402-CAP" value="0u1" x="124.9396" y="20.9496" rot="MR0">
 <attribute name="PARTNO" value="C0603C222J5RACTU" x="124.9396" y="20.9496" size="1.778" layer="28" rot="MR0" display="off"/>
 </element>
