File: PXF_CAPE_PCB/PixHawk_Fire_v1.3.brd (EAGLE design)
At the start: 86.4 x 54.6 mm, 239 parts, among them J305 DF13-3P-1.25V, J306 DF13-4P-1.25V, J307 DF13-4P-1.25V, J308 DF13-4P-1.25V, J309 DF13-5P-1.25V, J310 DF13-4P-1.25V, J314 DF13-4P-1.25V, J701 JST-ZH-3, J801 DF13C-6P-1.25V, M3_MOUNT901 MOUNT-HOLE3.1MM, M3_MOUNT902 MOUNT-HOLE3.1MM, M3_MOUNT903 MOUNT-HOLE3.1MM, M3_MOUNT904 MOUNT-HOLE3.1MM, Q501 MMBT3906LT1SMD, U1 EEPROM-I2CSMD, U102 FM25V01, U2 EEPROM-I2CSMD, U201 TXS0108QFN20, U202 TXS0108QFN20, U301 MAX3051, U302 TXS0108QFN20, U303 PCA9306, U401 MS5611-01BA, U402 MS5611-01BA, U403 MPU-6000, U405 MPU-9250, U406 LSM9DS0LSM9DS0, U407 BMP280_PRELIM, U501 BQ24315, U502 MIC5332, U503 BQ24315, U601 TCA62724FMG, U602 LT3469, U603 LRTB GFTG-T7AW-1+V7A7-29+R5T9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, U701 TXS0108QFN20, U703 74LVC2G240, U704 BBB_3X14_RA, U801 BQ24313, U802 MIC5332, X801 4 pin head

Commit message: MPU6500 instead of MPU9250
MPU9250 replacement for MPU6500. Minimal changes have been done: C411
and C415 value change to .1uF. Model change of both Cs in order to
fulfill X7R and 10% type requeriments.
Parts:
- C411: value 2200p -> 0.1uF
- U405: value MPU-9250 -> MPU-6500
Changed lines of the file:
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@@
 <?xml version="1.0" encoding="utf-8"?>
 <!DOCTYPE eagle SYSTEM "eagle.dtd">
-<eagle version="6.4">
+<eagle version="6.6.0">
 <drawing>
 <settings>
@@
 <grid distance="0.5" unitdist="mil" unit="mil" style="lines" multiple="2" display="yes" altdistance="0.003125" altunitdist="mic" altunit="mm"/>
 <layers>
-<layer number="1" name="Top" color="4" fill="1" visible="no" active="yes"/>
+<layer number="1" name="Top" color="4" fill="1" visible="yes" active="yes"/>
 <layer number="2" name="Ground" color="2" fill="10" visible="no" active="yes"/>
 <layer number="3" name="Horizontal" color="13" fill="15" visible="no" active="yes"/>
@@
 <layer number="12" name="Route12" color="1" fill="5" visible="no" active="no"/>
 <layer number="13" name="Route13" color="4" fill="5" visible="no" active="no"/>
-<layer number="14" name="Vertical" color="14" fill="1" visible="no" active="yes"/>
+<layer number="14" name="Vertical" color="14" fill="1" visible="yes" active="yes"/>
 <layer number="15" name="Power" color="11" fill="15" visible="no" active="yes"/>
-<layer number="16" name="Bottom" color="1" fill="1" visible="no" active="yes"/>
-<layer number="17" name="Pads" color="2" fill="1" visible="no" active="yes"/>
-<layer number="18" name="Vias" color="2" fill="1" visible="no" active="yes"/>
+<layer number="16" name="Bottom" color="1" fill="1" visible="yes" active="yes"/>
+<layer number="17" name="Pads" color="2" fill="1" visible="yes" active="yes"/>
+<layer number="18" name="Vias" color="2" fill="1" visible="yes" active="yes"/>
 <layer number="19" name="Unrouted" color="13" fill="1" visible="no" active="yes"/>
 <layer number="20" name="Dimension" color="15" fill="1" visible="yes" active="yes"/>
-<layer number="21" name="tPlace" color="7" fill="1" visible="yes" active="yes"/>
-<layer number="22" name="bPlace" color="7" fill="1" visible="no" active="yes"/>
-<layer number="23" name="tOrigins" color="15" fill="1" visible="yes" active="yes"/>
-<layer number="24" name="bOrigins" color="15" fill="1" visible="no" active="yes"/>
-<layer number="25" name="tNames" color="7" fill="1" visible="yes" active="yes"/>
-<layer number="26" name="bNames" color="7" fill="1" visible="no" active="yes"/>
-<layer number="27" name="tValues" color="7" fill="1" visible="yes" active="yes"/>
-<layer number="28" name="bValues" color="7" fill="1" visible="no" active="yes"/>
+<layer number="21" name="tPlace" color="7" fill="1" visible="no" active="yes"/>
+<layer number="22" name="bPlace" color="7" fill="1" visible="yes" active="yes"/>
+<layer number="23" name="tOrigins" color="15" fill="1" visible="no" active="yes"/>
+<layer number="24" name="bOrigins" color="15" fill="1" visible="yes" active="yes"/>
+<layer number="25" name="tNames" color="7" fill="1" visible="no" active="yes"/>
+<layer number="26" name="bNames" color="7" fill="1" visible="yes" active="yes"/>
+<layer number="27" name="tValues" color="7" fill="1" visible="no" active="yes"/>
+<layer number="28" name="bValues" color="7" fill="1" visible="yes" active="yes"/>
 <layer number="29" name="tStop" color="7" fill="3" visible="no" active="yes"/>
 <layer number="30" name="bStop" color="7" fill="6" visible="no" active="yes"/>
@@
 <attribute name="PARTNO" value="0512811094" x="121.7322" y="13.4388" size="1.778" layer="27" rot="R180" display="off"/>
 </element>
-<element name="U405" library="pixhawk2" package="MPU-6500" value="MPU-9250" x="119.1738" y="27.0556" rot="MR0">
-<attribute name="PARTNO" value="MPU-9250" x="119.1738" y="27.0556" size="1.778" layer="28" rot="MR0" display="off"/>
+<element name="U405" library="pixhawk2" package="MPU-6500" value="MPU-6500" x="119.1738" y="27.0556" rot="MR0">
+<attribute name="PARTNO" value="MPU-6500" x="119.1738" y="27.0556" size="1.778" layer="28" rot="MR0" display="off"/>
+<attribute name="DATASHEET" value="http://www.invensense.com/mems/gyro/documents/PS-MPU-6500A-01.pdf" x="119.1738" y="27.0556" size="1.778" layer="28" rot="MR0" display="off"/>
 </element>
 <element name="C410" library="pixhawk2" package="0603-CAP" value="10n" x="120.4364" y="23.3324" rot="MR270">
@@
 </element>
 <element name="C415" library="pixhawk2" package="0402-CAP" value="u1F" x="122.1676" y="24.9208" rot="MR180">
-<attribute name="PARTNO" value="CC0402ZRY5V7BB104" x="122.1676" y="24.9208" size="1.778" layer="28" rot="MR180" display="off"/>
-</element>
-<element name="C411" library="pixhawk2" package="0603-CAP" value="2200p" x="118.9984" y="22.7924" rot="MR270">
-<attribute name="PARTNO" value="C0603C222J5RACTU" x="118.9984" y="22.7924" size="1.778" layer="28" rot="MR270" display="off"/>
+<attribute name="PARTNO" value="06034C104KAT2A" x="122.1676" y="24.9208" size="1.778" layer="28" rot="MR180" display="off"/>
+</element>
+<element name="C411" library="pixhawk2" package="0603-CAP" value="0.1uF" x="118.9984" y="22.7924" rot="MR270">
+<attribute name="PARTNO" value="06034C104KAT2A" x="118.9984" y="22.7924" size="1.778" layer="28" rot="MR270" display="off"/>
 </element>
 <element name="JP401" library="pixhawk2" package="SJ_3_0603_PASTE1&amp;2" value="JUMPER-30603" x="109.474" y="17.526" rot="R270">
