File: PXF_CAPE_PCB/PixHawk_Fire_v1.4.brd (EAGLE design)
At the start: 86.4 x 54.6 mm, 242 parts, among them J305 DF13-3P-1.25V, J306 DF13-4P-1.25V, J307 DF13-4P-1.25V, J308 DF13-4P-1.25V, J309 DF13-5P-1.25V, J310 DF13-4P-1.25V, J314 DF13-4P-1.25V, J701 JST-ZH-3, J801 DF13C-6P-1.25V, M3_MOUNT901 MOUNT-HOLE3.1MM, M3_MOUNT902 MOUNT-HOLE3.1MM, M3_MOUNT903 MOUNT-HOLE3.1MM, M3_MOUNT904 MOUNT-HOLE3.1MM, Q501 MMBT3906LT1SMD, U1 EEPROM-I2CSMD, U102 FM25V01, U2 EEPROM-I2CSMD, U201 TXS0108QFN20, U202 TXS0108QFN20, U301 MAX3051, U302 TXS0108QFN20, U303 PCA9306, U401 MS5611-01BA, U402 MS5611-01BA, U403 MPU-6000, U405 MPU-9250, U406 LSM9DS0LSM9DS0, U407 BMP280_PRELIM, U501 BQ24315, U502 MIC5332, U503 BQ24315, U601 TCA62724FMG, U602 LT3469, U603 LRTB GFTG-T7AW-1+V7A7-29+R5T9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, U701 TXS0108QFN20, U702 TXS0108QFN20, U703 74LVC2G240, U704 BBB_3X14_RA, U801 BQ24313, U802 MIC5332, X801 4 pin head

Commit message: Version 1.4, LSM9D -> MPU9255 change
Parts:
- removed C407: 10u/10V, pixhawk2:0805-CAP
- removed C408, C703: 0u1, pixhawk2:0402-CAP
- removed R718: 10K, pixhawk2:0402-RES
- removed U406: LSM9DS0LSM9DS0, pixhawk2:LSM9DS0
- removed U702: TXS0108QFN20, pixhawk2:QFN20-RGY
- added U404: MPU-9255, pixhawk2:MPU-6500
- C402: value 4.7u -> 10nF
- C403: value 0.22u -> 0.1uF
- C405: value 0u1 -> 2u2F
- C406: value 10u -> 0.1uF; device pixhawk2:0603-CAP -> pixhawk2:0402-CAP
- C409, C414: value 2200p -> 0u1
- C411: value 2200p -> 0.1uF
- U405: value MPU-9250 -> MPU-9255
- moved C403 4.60 mm to (112.7, 22.2), turned to 90 degrees
Connections:
- net !ACCEL_MAG_CS renamed SPI_0_!MPU_CS
- net MPU_6500_DRDY renamed MPU_9255_1_DRDY
- removed net !ACCEL_MAG_CS_INT: JP402.1, U406.20
- removed net CH_10_OUT: R707.P$1, U702.17
- removed net CH_11_OUT: R708.P$1, U702.18
- removed net CH_12_OUT: R709.P$1, U702.20
- removed net CH_5_OUT: R702.P$1, U702.12
- removed net CH_6_OUT: R703.P$1, U702.13
- removed net CH_7_OUT: R704.P$1, U702.14
- removed net CH_8_OUT: R705.P$1, U702.15
- removed net CH_9_OUT: R706.P$1, U702.16
- removed net GYRO_DRDY: FPC_401.5, U$101.34, U406.12
- removed net N$16: C403.P$1, U406.8
- removed net N$87: R204.P$1, U201.13
- removed net N$88: R211.P$1, U201.12
- new net MPU_9255_0_DRDY: FPC_401.5, U$101.34, U404.12
- new net SPI_0_!MPU_CS_INT: JP402.1, U404.19
- net !GYRO_CS_INT: no longer U406.19
- net ACCEL_DRDY: no longer U406.14
- net BBB-VDD_3V3: no longer C703.P$1, R718.P$2, U702.10, U702.19, U702.2
- net CH_10: now also R707.P$1; no longer U702.4
- net CH_11: now also R708.P$1; no longer U702.3
- net CH_12: now also R709.P$1; no longer U702.1
- net CH_5: now also R702.P$1; no longer U702.9
- net CH_6: now also R703.P$1; no longer U702.8
- net CH_7: now also R704.P$1; no longer U702.7
- net CH_8: now also R705.P$1; no longer U702.6
- net CH_9: now also R706.P$1; no longer U702.5
- net GND: now also C403.P$1, U404.11, U404.18, U404.20; no longer C407.P$2, C408.P$2, C703.P$2, R718.P$1, U406.1, U406.2, U406.3, U406.4, U406.5, U406.6, U702.11
- net MAG_DRDY: no longer U406.13
- net N$14: now also U404.10; no longer U406.9
- net N$8: now also U404.1, U404.8; no longer U406.7
- net SPI_0_MISO: now also U404.9; no longer U406.22
- net SPI_0_MOSI: now also U404.24; no longer U406.23
- net SPI_0_SCK: now also U404.23; no longer U406.21
- net USART4_CTS: now also R211.P$1
- net USART4_RTS: now also R204.P$1
- net VDD_3V3_SENSORS: now also U404.13, U405.1; no longer C407.P$1, C408.P$1, U406.18
Routing:
- net MPU_9255_0_DRDY: track 0.00 -> 44.6 mm, vias 0 -> 5
- net GYRO_DRDY: track 43.5 -> 0.00 mm, vias 5 -> 0
- net SPI_0_!MPU_CS_INT: track 0.00 -> 15.1 mm, vias 0 -> 1
- net !ACCEL_MAG_CS_INT: track 12.0 -> 0.00 mm, vias 1 -> 0
- net CH_5: track 31.2 -> 21.1 mm
- net GND: track 460.9 -> 452.3 mm, vias 68 -> 66
- net MAG_DRDY: track 48.5 -> 40.0 mm, vias 4 -> 3
- net SPI_0_!MPU_CS: track 41.3 -> 49.7 mm, vias 6 -> 8
- net SPI_0_MISO: track 61.9 -> 70.3 mm, vias 8 -> 7
- net CH_5_OUT: track 8.09 -> 0.00 mm
- net CH_12_OUT: track 7.66 -> 0.00 mm
- net CH_6: track 30.1 -> 22.8 mm
- net BBB-VDD_3V3: track 168.6 -> 161.3 mm, vias 20 -> 19
- net CH_6_OUT: track 6.40 -> 0.00 mm
- net SPI_0_MOSI: track 64.6 -> 71.0 mm
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Other:
- board text added: "(c)2014 Erle,PR,LM,3DR,AT,BN,AP"
- board text added: "PixHawk-Fire v1.2"
- board text added: "PixHawk-Fire v1.3"
- board text removed: "(c)2014 PR,LM,3DR,AT,BN,AP"
- board text removed: "PixHawk-Fire v1.0"
- board text removed: "Spek"
