File: PXF_CAPE_PCB/PixHawk_Fire_v1.4.sch (EAGLE design)
At the start: 242 parts, among them J305 DF13-3P-1.25V, J306 DF13-4P-1.25V, J307 DF13-4P-1.25V, J308 DF13-4P-1.25V, J309 DF13-5P-1.25V, J310 DF13-4P-1.25V, J314 DF13-4P-1.25V, J701 JST-ZH-3, J801 DF13C-6P-1.25V, M3_MOUNT901 MOUNT-HOLE3.1MM, M3_MOUNT902 MOUNT-HOLE3.1MM, M3_MOUNT903 MOUNT-HOLE3.1MM, M3_MOUNT904 MOUNT-HOLE3.1MM, Q501 MMBT3906LT1SMD, U1 EEPROM-I2CSMD, U102 FM25V01, U2 EEPROM-I2CSMD, U201 TXS0108QFN20, U202 TXS0108QFN20, U301 MAX3051, U302 TXS0108QFN20, U303 PCA9306, U401 MS5611-01BA, U402 MS5611-01BA, U403 MPU-6000, U405 MPU-9250, U406 LSM9DS0LSM9DS0, U407 BMP280_PRELIM, U501 BQ24315, U502 MIC5332, U503 BQ24315, U601 TCA62724FMG, U602 LT3469, U603 LRTB GFTG-T7AW-1+V7A7-29+R5T9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, U701 TXS0108QFN20, U702 TXS0108QFN20, U703 74LVC2G240, U704 BBB_3X14_RA, U801 BQ24313, U802 MIC5332, X801 4 pin head

Commit message: Version 1.4, LSM9D -> MPU9255 change
Parts:
- removed C407: 10u/10V, pixhawk2:CAP0805
- removed C408, C703: 0u1, pixhawk2:CAP0402
- removed R718: 10K, pixhawk2:RESISTOR0402-RES
- removed U406: LSM9DS0LSM9DS0, pixhawk2:LSM9DS0LSM9DS0
- removed U702: TXS0108QFN20, pixhawk2:TXS0108QFN20
- added U404: MPU-9255, pixhawk2:MPU-6500
- C402: value 4.7u -> 10nF; PARTNO C1608X7S1A475K080AC -> C0603C103J5RAC7411
- C403: value 0.22u -> 0.1uF; PARTNO CL10B224JP8NNNC -> C0603C222J5RACTU
- C405: value 0u1 -> 2u2F; BOM (none) -> EXCLUDE; PARTNO CL10B104JO8NNNC -> (none)
- C406: value 10u -> 0.1uF; device pixhawk2:CAP0603 -> pixhawk2:CAP0402; PARTNO C1608X7S0J106M080AC -> CC0402ZRY5V7BB104
- C409, C414: PARTNO C0603C222J5RACTU -> C0603C104K4RACTU
- C411: value 2200p -> 0.1uF
- U405: value MPU-9250 -> MPU-9255
Connections:
- net !ACCEL_MAG_CS renamed SPI_0_!MPU_CS
- net MPU_6500_DRDY renamed MPU_9255_1_DRDY
- removed net !ACCEL_MAG_CS_INT: JP402.1, U406.CS_XM
- removed net CH_10_OUT: R707.1, U702.B3
- removed net CH_11_OUT: R708.1, U702.B2
- removed net CH_12_OUT: R709.1, U702.B1
- removed net CH_5_OUT: R702.1, U702.B8
- removed net CH_6_OUT: R703.1, U702.B7
- removed net CH_7_OUT: R704.1, U702.B6
- removed net CH_8_OUT: R705.1, U702.B5
- removed net CH_9_OUT: R706.1, U702.B4
- removed net GYRO_DRDY: FPC_401G$5.S, U$101.GPOI2[17]_34, U406.DRDY_G
- removed net N$16: C403.1, U406.SETC_XM
- removed net N$87: R204.1, U201.B7
- removed net N$88: R211.1, U201.B8
- new net MPU_9255_0_DRDY: FPC_401G$5.S, U$101.GPOI2[17]_34, U404.INT
- new net SPI_0_!MPU_CS_INT: JP402.1, U404.RESV@2
- net !GYRO_CS_INT: no longer U406.CS_G
- net ACCEL_DRDY: no longer U406.INT2_XM
- net BBB-VDD_3V3: no longer C703.1, R718.2, U702.OE, U702.VCCA, U702.VCCB
- net CH_10: now also R707.1; no longer U702.A3
- net CH_11: now also R708.1; no longer U702.A2
- net CH_12: now also R709.1; no longer U702.A1
- net CH_5: now also R702.1; no longer U702.A8
- net CH_6: now also R703.1; no longer U702.A7
- net CH_7: now also R704.1; no longer U702.A6
- net CH_8: now also R705.1; no longer U702.A5
- net CH_9: now also R706.1; no longer U702.A4
- net GND: now also C403.1, U404.FSYNC, U404.GND, U404.RESV@1; no longer C407.2, C408.2, C703.2, R718.1, U406.GND@1, U406.GND@2, U406.GND@3, U406.GND@4, U406.GND@5, U406.NC, U702.GND
- net MAG_DRDY: no longer U406.INT1_XM
- net N$14: now also U404.REGOUT; no longer U406.SETP_XM
- net N$8: now also U404.NC@1, U404.VDDIO; no longer U406.C1_XM
- net SPI_0_MISO: now also U404.AD0/SDO; no longer U406.SDO_G, U406.SDO_XM
- net SPI_0_MOSI: now also U404.SDA/SDI; no longer U406.SDA
- net SPI_0_SCK: now also U404.SCL/SCLK; no longer U406.SPC
- net USART4_CTS: now also R211.1
- net USART4_RTS: now also R204.1
- net VDD_3V3_SENSORS: now also U404.VDD, U405.NC@1; no longer C407.1, C408.1, U406.VDD_IO
Other:
- note added: "Fix has been applied in the layout that short circuits VDD_5V and VDD_5V_BRICK"
- note added: "Issue#3: As the voltage translator U702 is not use, it has been erased"
- note removed: "ADD WIRE CONNECTING PIN 15, 16, 17 AND 18"
- note removed: "REMOVE CONNECTION FROM PIN 1 TO GND BY CUTTING TRACE ON PCB"
- moved on the sheet: C402, C403, C405, C406, C410, C411, U405
